Commit message: Added Random Button Pose

File: kortex_bringup/world/warehouse.sdf.xacro (robot description, xacro)
@@ -1,18 +1,22 @@
-<?xml version="1.0" ?>
-<!-- =================================================================================== -->
-<!-- |    This document was autogenerated by xacro from /home/rafilappy/ws_moveit/install/kortex_bringup/share/kortex_bringup/world/warehouse.sdf.xacro | -->
-<!-- |    EDITING THIS FILE BY HAND IS NOT RECOMMENDED                                 | -->
-<!-- =================================================================================== -->
-<sdf version="1.7">
-  <world name="warehouse">
+<?xml version='1.0' encoding='ASCII'?>
+<sdf version='1.7' xmlns:xacro="http://www.ros.org/wiki/xacro">
+  <world name='warehouse'>
+    <xacro:arg name="btn_x" default="0.5"/>
+    <xacro:arg name="btn_y" default="0.0"/>
+    <xacro:arg name="btn_z" default="0.0"/>
+    <xacro:arg name="btn_roll" default="0.0"/>
+    <xacro:arg name="btn_pitch" default="0.0"/>
+    <xacro:arg name="btn_yaw" default="0.0"/>
     <physics type="ode">
-      <update_rate>1000</update_rate>
+    <update_rate>1000</update_rate>
       <max_step_size>0.001</max_step_size>
       <real_time_factor>1.0</real_time_factor>
     </physics>
-    <plugin filename="libignition-gazebo-physics-system.so" name="ignition::gazebo::systems::Physics"/>
-    <plugin filename="libignition-gazebo-user-commands-system.so" name="ignition::gazebo::systems::UserCommands"/>
-    <plugin filename="libignition-gazebo-scene-broadcaster-system.so" name="ignition::gazebo::systems::SceneBroadcaster"/>
-    <plugin filename="libignition-gazebo-sensors-system.so" name="ignition::gazebo::systems::Sensors">
+    <plugin name='ignition::gazebo::systems::Physics' filename='libignition-gazebo-physics-system.so'/>
+    <plugin name='ignition::gazebo::systems::UserCommands' filename='libignition-gazebo-user-commands-system.so'/>
+    <plugin name='ignition::gazebo::systems::SceneBroadcaster' filename='libignition-gazebo-scene-broadcaster-system.so'/>
+   <plugin
+      filename="libignition-gazebo-sensors-system.so"
+      name="ignition::gazebo::systems::Sensors">
       <render_engine>ogre2</render_engine>
     </plugin>
@@ -31,8 +35,8 @@
       <direction>0 0 -1</direction>
     </light> -->
-    <model name="ground_plane">
+    <model name='ground_plane'>
       <static>true</static>
-      <link name="link">
-        <collision name="collision">
+      <link name='link'>
+        <collision name='collision'>
           <geometry>
             <plane>
@@ -63,11 +67,11 @@
       <static>true</static>
     </include> -->
-    <include>
-      <uri>
+<include>
+  <uri>
   https://fuel.gazebosim.org/1.0/rahgirafi/models/Push to open button
   </uri>
-      <name>Push_to_Open_Button</name>
-      <pose>0.5 0.5315276018847506 0.6348655397882627 0.0 0.0 0.0</pose>
-    </include>
+  <name>Push_to_Open_Button</name>
+  <pose>$(arg btn_x) $(arg btn_y) $(arg btn_z) $(arg btn_roll) $(arg btn_pitch) $(arg btn_yaw)</pose>
+</include>
     <!-- Shelves -->
     <include>
