Commit message: made some necessary changes for flawless simulation into the srdf, yaml,rviz, launch files

File: kortex_description/arms/gen3/7dof/urdf/gen3_macro.xacro (robot description, xacro)
@@ -173,5 +173,5 @@
       <axis
         xyz="0 0 1" />
-      <limit lower="-2.24" upper="2.24" effort="39" velocity="1.3963" />
+      <limit lower="-2.27" upper="2.27" effort="39" velocity="1.3963" />
     </joint>
     <link name="${prefix}half_arm_2_link">
@@ -263,5 +263,5 @@
       <axis
         xyz="0 0 1" />
-      <limit lower="-2.57" upper="2.57" effort="39" velocity="1.3963" />
+      <limit lower="-2.60" upper="2.60" effort="39" velocity="1.3963" />
     </joint>
     <link name="${prefix}spherical_wrist_1_link">
@@ -353,5 +353,5 @@
       <axis
         xyz="0 0 1" />
-      <limit lower="-2.09" upper="2.09" effort="9" velocity="1.2218" />
+      <limit lower="-2.12" upper="2.12" effort="9" velocity="1.2218" />
     </joint>
     <xacro:if value="${vision}">
