Commit message: Integrated Realsense Camera

File: kortex_description/arms/gen3/6dof/urdf/gen3_macro.xacro (robot description, xacro)
@@ -22,5 +22,5 @@
     gripper_max_force:=100.0
     use_fake_hardware:=false
-    fake_sensor_commands:=false
+    mock_sensor_commands:=false
     sim_gazebo:=false
     sim_ignition:=false
@@ -36,5 +36,5 @@
       name="${prefix}KortexMultiInterfaceHardware" prefix="${prefix}"
       use_fake_hardware="${use_fake_hardware}"
-      fake_sensor_commands="${fake_sensor_commands}"
+      mock_sensor_commands="${mock_sensor_commands}"
       sim_gazebo="${sim_gazebo}"
       sim_ignition="${sim_ignition}"

File: kortex_description/arms/gen3/6dof/urdf/kortex.ros2_control.xacro (robot description, xacro)
@@ -5,5 +5,5 @@
     prefix
     use_fake_hardware:=false
-    fake_sensor_commands:=false
+    mock_sensor_commands:=false
     sim_gazebo:=false
     sim_ignition:=false
@@ -40,5 +40,5 @@
         <xacro:if value="${use_fake_hardware}">
           <plugin>mock_components/GenericSystem</plugin>
-          <param name="fake_sensor_commands">${fake_sensor_commands}</param>
+          <param name="mock_sensor_commands">${mock_sensor_commands}</param>
           <param name="state_following_offset">0.0</param>
         </xacro:if>

File: kortex_description/arms/gen3/7dof/urdf/gen3_macro.xacro (robot description, xacro)
@@ -22,5 +22,5 @@
     gripper_max_force:=100.0
     use_fake_hardware:=false
-    fake_sensor_commands:=false
+    mock_sensor_commands:=false
     sim_gazebo:=false
     sim_ignition:=false
@@ -33,9 +33,11 @@
     <!-- ros2 control include -->
     <xacro:include filename="$(find kortex_description)/arms/gen3/${dof}dof/urdf/kortex.ros2_control.xacro" />
+    <xacro:include filename="$(find realsense2_description)/urdf/_d435.urdf.xacro" />
+    <xacro:property name="PI" value="3.1415926535897931"/>
     <xacro:kortex_ros2_control
       name="${prefix}KortexMultiInterfaceHardware"
       prefix="${prefix}"
       use_fake_hardware="${use_fake_hardware}"
-      fake_sensor_commands="${fake_sensor_commands}"
+      mock_sensor_commands="${mock_sensor_commands}"
       sim_gazebo="${sim_gazebo}"
       sim_ignition="${sim_ignition}"
@@ -401,4 +403,35 @@
     </link>
     </xacro:unless>
+    <xacro:sensor_d435 parent="${prefix}bracelet_link" name="${prefix}d435" use_nominal_extrinsics="true">
+      <origin xyz="0 0.05 0" rpy="0 ${PI/2} ${PI/2}"/>
+    </xacro:sensor_d435>
+    <link name="${prefix}d435_link_optical"></link>
+    <joint name="${prefix}d435_optical_joint" type="fixed">
+      <origin xyz="0 0 0" rpy="0 0 0" />
+      <parent link="${prefix}d435_link" />
+      <child  link="${prefix}d435_link_optical" />
+    </joint>
+    <gazebo reference="${prefix}d435_link">
+      <sensor name="${prefix}d435_camera" type="rgbd_camera">
+        <camera>
+          <horizontal_fov>1.25</horizontal_fov>
+          <image>
+            <width>640</width>
+            <height>480</height>
+          </image>
+          <clip>
+            <near>0.3</near>
+            <far>100</far>
+          </clip>
+          <gz_frame_id>${prefix}d435</gz_frame_id>
+          <optical_frame_id>${prefix}d435_link_optical</optical_frame_id>
+        </camera>
+        <always_on>1</always_on>
+        <update_rate>30</update_rate>
+        <visualize>true</visualize>
+        <gz_frame_id>${prefix}d435</gz_frame_id>
+        <topic>${prefix}/sensors/${prefix}d435_camera</topic>
+      </sensor>
+    </gazebo>
     <xacro:if value="${use_external_cable}">
       <joint

File: kortex_description/arms/gen3/7dof/urdf/kortex.ros2_control.xacro (robot description, xacro)
@@ -5,5 +5,5 @@
     prefix
     use_fake_hardware:=false
-    fake_sensor_commands:=false
+    mock_sensor_commands:=false
     sim_gazebo:=false
     sim_ignition:=false
@@ -40,5 +40,5 @@
         <xacro:if value="${use_fake_hardware}">
           <plugin>mock_components/GenericSystem</plugin>
-          <param name="fake_sensor_commands">${fake_sensor_commands}</param>
+          <param name="mock_sensor_commands">${mock_sensor_commands}</param>
           <param name="state_following_offset">0.0</param>
         </xacro:if>

File: kortex_description/arms/gen3_lite/6dof/urdf/gen3_lite_macro.xacro (robot description, xacro)
@@ -21,5 +21,5 @@
     gripper_max_force:=100.0
     use_fake_hardware:=false
-    fake_sensor_commands:=false
+    mock_sensor_commands:=false
     sim_gazebo:=false
     sim_ignition:=false
@@ -53,5 +53,5 @@
       name="${ros2_control_name}" prefix="${prefix}"
       use_fake_hardware="${use_fake_hardware}"
-      fake_sensor_commands="${fake_sensor_commands}"
+      mock_sensor_commands="${mock_sensor_commands}"
       sim_gazebo="${sim_gazebo}"
       sim_ignition="${sim_ignition}"

File: kortex_description/arms/gen3_lite/6dof/urdf/kortex.ros2_control.xacro (robot description, xacro)
@@ -5,5 +5,5 @@
     prefix
     use_fake_hardware:=false
-    fake_sensor_commands:=false
+    mock_sensor_commands:=false
     sim_gazebo:=false
     sim_ignition:=false
@@ -47,5 +47,5 @@
           <xacro:unless value="${moveit_active}">
             <plugin>mock_components/GenericSystem</plugin>
-            <param name="fake_sensor_commands">${fake_sensor_commands}</param>
+            <param name="mock_sensor_commands">${mock_sensor_commands}</param>
             <param name="state_following_offset">0.0</param>
           </xacro:unless>

File: kortex_description/grippers/gen3_lite_2f/urdf/gen3_lite_2f.ros2_control.xacro (robot description, xacro)
@@ -4,5 +4,5 @@
         prefix
         use_fake_hardware:=false
-        fake_sensor_commands:=false
+        mock_sensor_commands:=false
         sim_ignition:=false
         sim_isaac:=false
@@ -34,5 +34,5 @@
                 <xacro:if value="${use_fake_hardware}">
                     <plugin>mock_components/GenericSystem</plugin>
-                    <param name="mock_sensor_commands">${fake_sensor_commands}</param>
+                    <param name="mock_sensor_commands">${mock_sensor_commands}</param>
                     <param name="state_following_offset">0.0</param>
                 </xacro:if>

File: kortex_description/grippers/gen3_lite_2f/urdf/gen3_lite_2f_macro.xacro (robot description, xacro)
@@ -6,5 +6,5 @@
     com_port
     use_fake_hardware:=false
-    fake_sensor_commands:=false
+    mock_sensor_commands:=false
     sim_ignition:=false
     sim_isaac:=false
@@ -29,5 +29,5 @@
         prefix="${prefix}"
         use_fake_hardware="${use_fake_hardware}"
-        fake_sensor_commands="${fake_sensor_commands}"
+        mock_sensor_commands="${mock_sensor_commands}"
         sim_ignition="${sim_ignition}"
         sim_isaac="${sim_isaac}"

File: kortex_description/grippers/robotiq_2f_140/urdf/robotiq_2f_140_macro.xacro (robot description, xacro)
@@ -5,5 +5,5 @@
     prefix
     use_fake_hardware:=false
-    fake_sensor_commands:=false
+    mock_sensor_commands:=false
     sim_ignition:=false
     sim_isaac:=false
@@ -26,5 +26,5 @@
         com_port="${com_port}"
         use_fake_hardware="${use_fake_hardware}"
-        fake_sensor_commands="${fake_sensor_commands}"
+        mock_sensor_commands="${mock_sensor_commands}"
         sim_ignition="${sim_ignition}"
         sim_isaac="${sim_isaac}"

File: kortex_description/grippers/robotiq_2f_85/urdf/robotiq_2f_85_macro.xacro (robot description, xacro)
@@ -5,5 +5,5 @@
     prefix
     use_fake_hardware:=false
-    fake_sensor_commands:=false
+    mock_sensor_commands:=false
     sim_ignition:=false
     sim_isaac:=false
@@ -26,5 +26,5 @@
         com_port="${com_port}"
         use_fake_hardware="${use_fake_hardware}"
-        fake_sensor_commands="${fake_sensor_commands}"
+        mock_sensor_commands="${mock_sensor_commands}"
         sim_ignition="${sim_ignition}"
         sim_isaac="${sim_isaac}"

File: kortex_description/robots/gen3.xacro (robot description, xacro)
@@ -21,5 +21,5 @@
     <xacro:arg name="prefix" default="" />
     <xacro:arg name="use_fake_hardware" default="false" />
-    <xacro:arg name="fake_sensor_commands" default="false" />
+    <xacro:arg name="mock_sensor_commands" default="false" />
     <xacro:arg name="use_internal_bus_gripper_comm" default="false" />
     <xacro:arg name="use_external_cable" default="false" />
@@ -49,5 +49,5 @@
         prefix="$(arg prefix)"
         use_fake_hardware="$(arg use_fake_hardware)"
-        fake_sensor_commands="$(arg fake_sensor_commands)"
+        mock_sensor_commands="$(arg mock_sensor_commands)"
         sim_gazebo="$(arg sim_gazebo)"
         sim_ignition="$(arg sim_ignition)"

File: kortex_description/robots/gen3_2f85.urdf (robot description, URDF)
Before this commit: robot gen3_, 31 links, 30 joints
Links:
- link wrist_mounted_camera_link: geometry collision box size=0.02005 0.099 0.023; visual mesh filename=file://$(find realsense2_description)/meshes/d415.stl

File: kortex_description/robots/gen3_lite_gen3_lite_2f.xacro (robot description, xacro)
@@ -21,5 +21,5 @@
     <xacro:arg name="prefix" default="" />
     <xacro:arg name="use_fake_hardware" default="false" />
-    <xacro:arg name="fake_sensor_commands" default="false" />
+    <xacro:arg name="mock_sensor_commands" default="false" />
     <xacro:arg name="use_internal_bus_gripper_comm" default="true" />
     <xacro:arg name="use_external_cable" default="false" />
@@ -46,5 +46,5 @@
         prefix="$(arg prefix)"
         use_fake_hardware="$(arg use_fake_hardware)"
-        fake_sensor_commands="$(arg fake_sensor_commands)"
+        mock_sensor_commands="$(arg mock_sensor_commands)"
         sim_gazebo="$(arg sim_gazebo)"
         sim_ignition="$(arg sim_ignition)"

File: kortex_description/robots/kinova.urdf.xacro (robot description, xacro)
@@ -21,5 +21,5 @@
   <xacro:arg name="use_internal_bus_gripper_comm" default="false" />
   <xacro:arg name="use_fake_hardware" default="false" />
-  <xacro:arg name="fake_sensor_commands" default="false" />
+  <xacro:arg name="mock_sensor_commands" default="false" />
   <xacro:arg name="sim_gazebo" default="false" />
   <xacro:arg name="sim_ignition" default="false" />
@@ -58,5 +58,5 @@
     prefix="$(arg prefix)"
     use_fake_hardware="$(arg use_fake_hardware)"
-    fake_sensor_commands="$(arg fake_sensor_commands)"
+    mock_sensor_commands="$(arg mock_sensor_commands)"
     sim_gazebo="$(arg sim_gazebo)"
     sim_ignition="$(arg sim_ignition)"
@@ -89,65 +89,4 @@
       </plugin>
     </gazebo>
-    <gazebo reference="camera_color_frame">
-      <sensor name="camera_sensor" type="rgbd_camera">
-        <camera>
-          <horizontal_fov>1.047</horizontal_fov>
-          <image>
-            <width>$(arg camera_width)</width>
-            <height>$(arg camera_height)</height>
-            <format>RGB_INT8</format>
-          </image>
-          <clip>
-            <near>0.1</near>
-            <far>5</far>
-          </clip>
-          <distortion>
-            <k1>0.0</k1>
-            <k2>0.0</k2>
-            <k3>0.0</k3>
-            <p1>0.0</p1>
-            <p2>0.0</p2>
-            <center>0.5 0.5</center>
-          </distortion>
-          <lens>
-            <intrinsics>
-              <fx>554.25469</fx>
-              <fy>554.25469</fy>
-              <cx>320.5</cx>
-              <cy>240.5</cy>
-              <s>0</s>
-            </intrinsics>
-            <!-- These need to match the intrinsics above or
-            Ignition will default to different default values -->
-            <projection>
-              <p_fx>554.25469</p_fx>
-              <p_fy>554.25469</p_fy>
-              <p_cx>320.5</p_cx>
-              <p_cy>240.5</p_cy>
-              <tx>0</tx>
-              <ty>0</ty>
-            </projection>
-          </lens>
-          <noise>
-            <type>gaussian</type>
-            <mean>0</mean>
-            <stddev>0.00</stddev>
-          </noise>
-          <depth_camera>
-            <clip>
-              <near>0.25</near>
-              <far>5</far>
-            </clip>
-          </depth_camera>
-          <optical_frame_id>color_optical_frame</optical_frame_id>
-        </camera>
-        <ignition_frame_id>camera_color_frame</ignition_frame_id>
-        <always_on>1</always_on>
-        <update_rate>$(arg camera_fps)</update_rate>
-        <visualize>true</visualize>
-        <topic>wrist_mounted_camera</topic>
-        <enable_metrics>false</enable_metrics>
-      </sensor>
-    </gazebo>
   </xacro:if>
 </robot>

File: kortex_description/robots/kortex_robot.xacro (robot description, xacro)
@@ -19,5 +19,5 @@
     use_internal_bus_gripper_comm:=false
     use_fake_hardware:=false
-    fake_sensor_commands:=false
+    mock_sensor_commands:=false
     sim_gazebo:=false
     sim_ignition:=false
@@ -48,5 +48,5 @@
       use_internal_bus_gripper_comm="${use_internal_bus_gripper_comm}"
       use_fake_hardware="${use_fake_hardware}"
-      fake_sensor_commands="${fake_sensor_commands}"
+      mock_sensor_commands="${mock_sensor_commands}"
       sim_gazebo="${sim_gazebo}"
       sim_ignition="${sim_ignition}"
@@ -80,5 +80,5 @@
         prefix="${prefix}"
         use_fake_hardware="${use_fake_hardware}"
-        fake_sensor_commands="${fake_sensor_commands}"
+        mock_sensor_commands="${mock_sensor_commands}"
         sim_ignition="${sim_ignition}"
         sim_isaac="${sim_isaac}"

Commit message: Changed the urdf to add gazebo sensors

File: kortex_description/arms/gen3/6dof/urdf/gen3_macro.xacro (robot description, xacro)
@@ -33,4 +33,5 @@
     <!-- ros2 control include -->
     <xacro:include filename="$(find kortex_description)/arms/gen3/${dof}dof/urdf/kortex.ros2_control.xacro" />
+    <xacro:include filename="$(find realsense2_description)/urdf/_d435.urdf.xacro" />
     <xacro:kortex_ros2_control
       name="${prefix}KortexMultiInterfaceHardware" prefix="${prefix}"
@@ -357,5 +358,5 @@
       <link name="${prefix}camera_link" />
       <joint name="${prefix}camera_module" type="fixed">
-        <origin xyz="0 0.05639 -0.00305" rpy="3.14159265358979 3.14159265358979 0" />
+        <origin xyz="0 0.05639 -0.00305" rpy="0 -1.5708 -1.5708" />
         <parent link="${prefix}end_effector_link" />
         <child  link="${prefix}camera_link" />
@@ -373,4 +374,29 @@
         <child  link="${prefix}camera_color_frame" />
       </joint>
+      <!-- Camera sensor for Ignition Gazebo simulation -->
+      <xacro:if value="${sim_ignition}">
+        <gazebo reference="${prefix}camera_link">
+          <sensor name="${prefix}camera_sensor" type="rgbd_camera">
+            <camera>
+              <horizontal_fov>1.25</horizontal_fov>
+              <image>
+                <width>640</width>
+                <height>480</height>
+              </image>
+              <clip>
+                <near>0.3</near>
+                <far>100</far>
+              </clip>
+              <gz_frame_id>${prefix}camera_link</gz_frame_id>
+              <optical_frame_id>${prefix}camera_color_frame</optical_frame_id>
+            </camera>
+            <always_on>1</always_on>
+            <update_rate>30</update_rate>
+            <visualize>true</visualize>
+            <gz_frame_id>${prefix}camera_link</gz_frame_id>
+            <topic>${prefix}/sensors/${prefix}camera</topic>
+          </sensor>
+        </gazebo>
+      </xacro:if>
     </xacro:if>
   </xacro:macro>

Commit message: Fixed camera frame

File: kortex_description/arms/gen3/6dof/urdf/gen3_macro.xacro (robot description, xacro)
@@ -364,5 +364,5 @@
       <link name="${prefix}camera_depth_frame" />
       <joint name="${prefix}depth_module" type="fixed">
-        <origin xyz="0.0275 0.066 -0.00305" rpy="3.14159265358979 3.14159265358979 0" />
+        <origin xyz="0.0275 0.066 -0.00305" rpy="0 1.5708 1.5708" />
         <parent link="${prefix}end_effector_link" />
         <child  link="${prefix}camera_depth_frame" />
@@ -389,5 +389,5 @@
               </clip>
               <gz_frame_id>${prefix}camera_link</gz_frame_id>
-              <optical_frame_id>${prefix}camera_color_frame</optical_frame_id>
+              <optical_frame_id>${prefix}camera_link</optical_frame_id>
             </camera>
             <always_on>1</always_on>
